Commit message: update confbot with mesh

File: confbot_description/urdf/confbot.urdf (robot description, URDF)
Before this commit: robot confbot, 4 links, 3 joints
Links:
- link base_link: geometry visual mesh filename=package://confbot_description/meshes/confbot.dae
- link wheel_l_link: geometry visual cylinder length=0.2 radius=0.3
- link wheel_r_link: geometry visual cylinder length=0.2 radius=0.3

Commit message: Gazebo support (draft) (#19)
* first step to gazebo support

rename links and joints to have semantic names
add inertia to all links
add laser and diffdrive plugins

Signed-off-by: Mikael Arguedas <mikael.arguedas@gmail.com>

* add scripts taken and modifies from turtlebot3_simulation

Signed-off-by: Mikael Arguedas <mikael.arguedas@gmail.com>

* add simulation launchfile

Signed-off-by: Mikael Arguedas <mikael.arguedas@gmail.com>

* move urdf_spawner back in confbot_simulation

Signed-off-by: Mikael Arguedas <mikael.arguedas@gmail.com>

* restore package:// path

Signed-off-by: Mikael Arguedas <mikael.arguedas@gmail.com>

* add dependencies not part of the nightly image

Signed-off-by: Mikael Arguedas <mikael.arguedas@gmail.com>

* blacklist dependencies built from source from the test invocation

Signed-off-by: Mikael Arguedas <mikael.arguedas@gmail.com>

* fix test failures

Signed-off-by: Mikael Arguedas <mikael.arguedas@gmail.com>

* almost empty world

Signed-off-by: Mikael Arguedas <mikael.arguedas@gmail.com>

* rebasing

Signed-off-by: Mikael Arguedas <mikael.arguedas@gmail.com>

* dont set use_sim_time as currently doesn't impact time used

Signed-off-by: Mikael Arguedas <mikael.arguedas@gmail.com>

* Revert "dont set use_sim_time as currently doesn't impact time used"

This reverts commit b79ca27fe72c74bf2c06e012c26e488e419ecee2.

* use libgazebo_ros_init to have sim time published

Signed-off-by: Mikael Arguedas <mikael.arguedas@gmail.com>

* fix conversion error from string to bool

Signed-off-by: Karsten Knese <karsten@openrobotics.org>

* actually using the sim time parameter correctly

Signed-off-by: Karsten Knese <karsten@openrobotics.org>

* interpret launch configuration as yaml

Signed-off-by: Karsten Knese <karsten@openrobotics.org>

* visualize the laser scan in gazebo

Signed-off-by: Karsten Knese <karsten@openrobotics.org>

* use sim time

Signed-off-by: Karsten Knese <karsten@openrobotics.org>

* make laser_frame point forward

Signed-off-by: Mikael Arguedas <mikael.arguedas@gmail.com>

* gazebo_ros now declares/set use_sim_time to true by default

Signed-off-by: Mikael Arguedas <mikael.arguedas@gmail.com>

* add camera

Need to create an optical frame to match REP103 as camera plugin uses x forward and not z
forward
Need to source Gazebo setup file manually for the camera plugin to be
found and loaded successfully
No namespace provided to plugin as it appends the sensor name to the
namespace already, otherwise results in
/confbot_camera/confobt_camera/image_raw

Signed-off-by: Mikael Arguedas <mikael.arguedas@gmail.com>

* move back camera_frame on the robot base

Signed-off-by: Mikael Arguedas <mikael.arguedas@gmail.com>

* add rviz config for gazebo

Signed-off-by: Mikael Arguedas <mikael.arguedas@gmail.com>

* add preliminary Gazebo section

Signed-off-by: Mikael Arguedas <mikael.arguedas@gmail.com>

* fix config file name in instructions

Signed-off-by: Mikael Arguedas <mikael.arguedas@gmail.com>

File: confbot_description/urdf/confbot.urdf (robot description, URDF)
Before this commit: robot confbot, 4 links, 3 joints
Links:
- removed link laser_link
- added link camera_frame, mass 1; collision box size=0.1 0.1 0.1
- added link camera_optical_frame
- added link caster_wheel_front_link, mass 1; collision sphere radius=0.05; visual sphere radius=0.05
- added link caster_wheel_rear_link, mass 1; collision sphere radius=0.05; visual sphere radius=0.05
- added link laser_frame, mass 1; collision box size=0.1 0.1 0.1; visual box size=0.1 0.1 0.1
- link base_link: mass None -> 5; geometry collision box size=1 1 0.1; visual mesh filename=package://confbot_description/meshes/confbot.dae
- link wheel_l_link: mass None -> 1; geometry collision cylinder length=0.05 radius=0.1; visual cylinder length=0.05 radius=0.1
- link wheel_r_link: mass None -> 1; geometry collision cylinder length=0.05 radius=0.1; visual cylinder length=0.05 radius=0.1
Joints:
- removed joint wheel_l_frame
- removed joint wheel_r_frame
- added joint camera_frame: type fixed, parent base_link, child camera_frame, origin xyz=0.4 0.0 0.2 rpy=0 0 0
- added joint camera_optical_fixed_joint: type fixed, parent camera_frame, child camera_optical_frame, origin xyz=0 0 0 rpy=0 1.57079632679 0
- added joint caster_wheel_front_joint: type continuous, parent base_link, child caster_wheel_front_link, origin xyz=0.4 0.0 -0.05 rpy=0 0 0, axis 1.0 1.0 0
- added joint caster_wheel_rear_joint: type continuous, parent base_link, child caster_wheel_rear_link, origin xyz=-0.4 0.0 -0.05 rpy=0 0 0, axis 1.0 1.0 0
- added joint wheel_l_joint: type continuous, parent base_link, child wheel_l_link, origin xyz=0 0.55 0.0 rpy=0 0 0, axis 0 1.0 0
- added joint wheel_r_joint: type continuous, parent base_link, child wheel_r_link, origin xyz=0 -0.55 0.0 rpy=0 0 0, axis 0 1.0 0
- joint laser_frame: child laser_link -> laser_frame; origin xyz=0.45 0.0 0.1 rpy=0 0 -1.57 -> xyz=0.45 0.0 0.1 rpy=0 0 0
